Commit message: fix(firmware,ros2,sdk): resolve 12 critical + 18 important issues from code review
CRITICAL fixes:
- firmware: Replace broken Ed25519/ECDSA OTA verification with ECDSA P-256
- firmware: Fix DTLS port collision (both UDP+DTLS bound to 8888), update header macro to 5684
- firmware: Fix zero-key validation using 32-byte buffer (was 16)
- firmware: Add portMUX_TYPE spinlock for safety_state_t atomicity across dual cores
- firmware: Add volatile qualifier to motor_control stopped flag
- firmware: Add I2C read error checking in payload_hotplug.c to prevent latch zeroing
- firmware: Validate EEPROM capabilities against hardware allowlist
- firmware: Add OTA image max size validation (16MB), handle UINT32_MAX version parse failure
- ros2: Remove double Nav2 launch in gazebo_nav.launch.py (was launching Nav2 twice)
- ros2: Fix URDF base_footprint_joint z-offset (was ground_clearance + wheel_radius, now wheel_radius)
- ros2: Remove software E-stop reset from EmergencyStop.srv (safety rule violation)
- sdk: Remove non-existent uses_usb attribute in hello_payload.py
- sdk: Fix onBattery this-binding lost in web_basic/main.js
- sdk: Fix CSS grid row/area count mismatch (4 tracks vs 5 areas)

IMPORTANT fixes:
- firmware: Remove default PSK credentials from dtls_transport.h public header
- firmware: Add i2c_bus mutex locking to imu.c and thermal_monitor.c
- firmware: Add RMT semaphore drain before each ultrasonic read
- ros2: Rename recoveries_server to behavior_server (Nav2 Humble+)
- ros2: Fix bridge_params.yaml world name mismatch with obstacles.sdf
- ros2: Fix IMU Gazebo sensor reference from base_link to imu_link
- ros2: Add missing tf2_ros and slam_toolbox exec_depend
- sdk: Add rAF throttle to sensor-radar.ts onRange updates
- sdk: Fix eeprom_validator.py import path for standalone execution
- sdk: Fix sensor_payload.py I2C bus leak on discover failure
- sdk: Align payload_protocol.py name encoding to ASCII (matches validator)
- sdk: Add E-stop reset confirmation dialog in web_basic
- docs: Fix E-stop GPIO number in firmware_flash.md (36 -> 41)
- hardware: Remove invalid CSV comment lines from BOM files

File: ros2_ws/robot_description/urdf/robot.urdf.xacro (robot description, xacro)
@@ -112,5 +112,5 @@
     <parent link="base_footprint"/>
     <child link="base_link"/>
-    <origin xyz="0 0 ${ground_clearance + wheel_radius}" rpy="0 0 0"/>
+    <origin xyz="0 0 ${wheel_radius}" rpy="0 0 0"/>
   </joint>
   <!-- Wheels -->

File: ros2_ws/robot_simulation/urdf/robot_gazebo.urdf.xacro (robot description, xacro)
@@ -119,5 +119,5 @@
   <!-- IMU Sensor Plugin                                                -->
   <!-- ================================================================ -->
-  <gazebo reference="base_link">
+  <gazebo reference="imu_link">
     <sensor name="imu_sensor" type="imu">
       <always_on>true</always_on>

Commit message: feat(hardware): enlarge Industrial SKU to 500x400mm chassis with 97mm wheels
- Add Kconfig chassis geometry menu (wheel radius, track width, wheelbase)
  with x10 integer trick for float precision
- Parameterize URDF with xacro:arg (defaults preserve Basic/Standard/Pro)
- Add OpaqueFunction SKU selection in robot.launch.py and gazebo.launch.py
- Create nav2_params_industrial.yaml (robot_radius=0.32, higher velocities)
- Update BOM: 97mm Mecanum wheels, 550 motor brackets, 500x400x100 enclosure
- Update hardware/structure docs with Industrial dimensions and load specs
- Add industrial/ DXF placeholder with expected drawing list
- Parameterize test_urdf.py for standard + industrial assertions
- Add TestNav2ParamsIndustrial test class

Firmware host tests (188), Python SDK (118), web_control vitest (41),
Playwright E2E (53), cross-layer validation — all passing.

File: ros2_ws/robot_description/urdf/robot.urdf.xacro (robot description, xacro)
@@ -2,15 +2,24 @@
 <!-- SPDX-License-Identifier: Apache-2.0 -->
 <robot xmlns:xacro="http://www.ros.org/wiki/xacro" name="robot_platform">
-  <!-- Parameters -->
-  <xacro:property name="chassis_length" value="0.300"/>
-  <xacro:property name="chassis_width" value="0.250"/>
-  <xacro:property name="chassis_height" value="0.080"/>
-  <xacro:property name="chassis_mass" value="2.5"/>
-  <xacro:property name="wheel_radius" value="0.024"/>
-  <xacro:property name="wheel_width" value="0.040"/>
-  <xacro:property name="wheel_mass" value="0.15"/>
-  <xacro:property name="wheelbase" value="0.180"/>
-  <xacro:property name="track_width" value="0.200"/>
-  <xacro:property name="ground_clearance" value="0.025"/>
+  <!-- SKU-configurable parameters (defaults = Basic/Standard/Pro) -->
+  <xacro:arg name="chassis_length" default="0.300"/>
+  <xacro:arg name="chassis_width" default="0.250"/>
+  <xacro:arg name="chassis_height" default="0.080"/>
+  <xacro:arg name="chassis_mass" default="2.5"/>
+  <xacro:arg name="wheel_radius" default="0.024"/>
+  <xacro:arg name="wheel_width" default="0.040"/>
+  <xacro:arg name="wheel_mass" default="0.15"/>
+  <xacro:arg name="wheelbase" default="0.180"/>
+  <xacro:arg name="track_width" default="0.200"/>
+  <xacro:property name="chassis_length" value="$(arg chassis_length)"/>
+  <xacro:property name="chassis_width" value="$(arg chassis_width)"/>
+  <xacro:property name="chassis_height" value="$(arg chassis_height)"/>
+  <xacro:property name="chassis_mass" value="$(arg chassis_mass)"/>
+  <xacro:property name="wheel_radius" value="$(arg wheel_radius)"/>
+  <xacro:property name="wheel_width" value="$(arg wheel_width)"/>
+  <xacro:property name="wheel_mass" value="$(arg wheel_mass)"/>
+  <xacro:property name="wheelbase" value="$(arg wheelbase)"/>
+  <xacro:property name="track_width" value="$(arg track_width)"/>
+  <xacro:property name="ground_clearance" value="${wheel_radius + 0.001}"/>
   <!-- Materials -->
   <material name="dark_grey">

File: ros2_ws/robot_simulation/urdf/robot_gazebo.urdf.xacro (robot description, xacro)
@@ -10,4 +10,14 @@
 -->
 <robot xmlns:xacro="http://www.ros.org/wiki/xacro" name="robot_platform_gazebo">
+  <!-- SKU-configurable parameters forwarded to base description -->
+  <xacro:arg name="chassis_length" default="0.300"/>
+  <xacro:arg name="chassis_width" default="0.250"/>
+  <xacro:arg name="chassis_height" default="0.080"/>
+  <xacro:arg name="chassis_mass" default="2.5"/>
+  <xacro:arg name="wheel_radius" default="0.024"/>
+  <xacro:arg name="wheel_width" default="0.040"/>
+  <xacro:arg name="wheel_mass" default="0.15"/>
+  <xacro:arg name="wheelbase" default="0.180"/>
+  <xacro:arg name="track_width" default="0.200"/>
   <!-- Include the base robot description -->
   <xacro:include filename="$(find robot_description)/urdf/robot.urdf.xacro"/>

Commit message: fix(hardware): resolve cross-layer hardware-software inconsistencies
CRITICAL fixes:
- CAN bus SPI pins reassigned from GPIO 33-37 (PSRAM-occupied on N8R8
  module) to GPIO 9-12,18 (freed by Industrial LiDAR replacing ultrasonics)
- Document GPIO 45/46 strapping pin PCB pull resistor requirements
- Add #ifdef guard for GPIO 4 dual assignment (ENC_RR_B vs BATT_PACK2_ADC)
- Fix ADC_ATTEN_DB_12 → ADC_ATTEN_DB_11 for ESP-IDF 5.x compatibility
- Guard CHARGE_ADC behind CONFIG_ROBOT_DOCKING_ENABLED to prevent GPIO 9
  conflict with US_ECHO_LEFT

HIGH fixes:
- Add Standard/Basic SKU xacro args to robot.launch.py (was only Industrial)
- Fix SDK battery thresholds to match firmware cell-voltage constants
- Add BTS7960 motor driver documentation for Industrial SKU pin mapping
- Correct ground clearance values (Standard: 35mm, Industrial: 52mm)

MEDIUM fixes:
- Add N20 1:50 motor entries to Standard BOM (were missing)
- Correct PBC-34 5V current rating from 5A to 3A (matches TPS5430DDAR)
- Update eeprom_validator MAX_5V_MA limit and warning threshold
- Fix host-side test comment claiming Basic defaults cover Standard SKU
- Use ground_clearance property in URDF base_footprint_joint (was unused)

File: ros2_ws/robot_description/urdf/robot.urdf.xacro (robot description, xacro)
@@ -121,5 +121,5 @@
     <parent link="base_footprint"/>
     <child link="base_link"/>
-    <origin xyz="0 0 ${wheel_radius}" rpy="0 0 0"/>
+    <origin xyz="0 0 ${ground_clearance}" rpy="0 0 0"/>
   </joint>
   <!-- Wheels -->

Commit message: feat(sdk,ros2): enhance mock backend, fix Gazebo bridge, polish PyPI release
Mock backend enhancements:
- Add scene-based obstacle layouts (office_v2, apartment_v1, corridor_v1, obstacles, empty)
- Implement ray-AABB intersection for LiDAR raycasting against obstacles
- Add circle-rect collision detection with incremental move stepping
- Add Gaussian sensor noise (σ=0.008m) matching real LD06 LiDAR
- New mock_scenes.py with 5 configurable environment presets

Gazebo bridge fixes:
- Add camera RGB/depth topic mappings to bridge_params.yaml
- Add aggregated /scan LiDAR topic bridge (GZ_TO_ROS)
- Add camera_info topic for intrinsics
- Add RGB camera sensor plugin (640x480, 30Hz) to URDF
- Add depth camera sensor plugin (640x480, 15Hz) to URDF
- Add 2D LiDAR sensor plugin (360 samples, 0.12-12m, 10Hz) to URDF
- Add camera_link and lidar_link to robot description URDF

PyPI release polish:
- Add Issues and Changelog URLs to pyproject.toml
- Add py.typed PEP 561 marker for type checker support
- Add keywords: simulation, deep-learning, gymnasium

Example defaults:
- Change vlm_navigation.py default backend from gazebo to mock
- Change data_collection.py default backend from gazebo to mock
- Add argparse to slam_exploration.py with mock as default backend

All 358 tests pass. Cross-layer validation scripts clean.

File: ros2_ws/robot_description/urdf/robot.urdf.xacro (robot description, xacro)
@@ -170,3 +170,49 @@
     <origin xyz="0 0 ${chassis_height + 0.005}" rpy="0 0 0"/>
   </joint>
+  <!-- Camera (fisheye 1080p, mounted on front upper chassis) -->
+  <link name="camera_link">
+    <visual>
+      <geometry>
+        <box size="0.025 0.025 0.025"/>
+      </geometry>
+      <material name="dark_grey"/>
+    </visual>
+    <collision>
+      <geometry>
+        <box size="0.025 0.025 0.025"/>
+      </geometry>
+    </collision>
+    <inertial>
+      <mass value="0.02"/>
+      <inertia ixx="0.000001" ixy="0" ixz="0" iyy="0.000001" iyz="0" izz="0.000001"/>
+    </inertial>
+  </link>
+  <joint name="camera_joint" type="fixed">
+    <parent link="base_link"/>
+    <child link="camera_link"/>
+    <origin xyz="${chassis_length/2 - 0.01} 0 ${chassis_height + 0.015}" rpy="0 0 0"/>
+  </joint>
+  <!-- 2D LiDAR (LD06, mounted on top center) -->
+  <link name="lidar_link">
+    <visual>
+      <geometry>
+        <cylinder radius="0.035" length="0.020"/>
+      </geometry>
+      <material name="dark_grey"/>
+    </visual>
+    <collision>
+      <geometry>
+        <cylinder radius="0.035" length="0.020"/>
+      </geometry>
+    </collision>
+    <inertial>
+      <mass value="0.05"/>
+      <inertia ixx="0.000002" ixy="0" ixz="0" iyy="0.000002" iyz="0" izz="0.000003"/>
+    </inertial>
+  </link>
+  <joint name="lidar_joint" type="fixed">
+    <parent link="base_link"/>
+    <child link="lidar_link"/>
+    <origin xyz="0 0 ${chassis_height + 0.012}" rpy="0 0 0"/>
+  </joint>
 </robot>

File: ros2_ws/robot_simulation/urdf/robot_gazebo.urdf.xacro (robot description, xacro)
@@ -318,3 +318,97 @@
     </sensor>
   </gazebo>
+  <!-- ================================================================ -->
+  <!-- Camera Sensor — RGB + Depth for VLM/VLA vision tasks             -->
+  <!-- ================================================================ -->
+  <gazebo reference="camera_link">
+    <material>
+      <ambient>0.2 0.2 0.2 1.0</ambient>
+      <diffuse>0.25 0.25 0.25 1.0</diffuse>
+    </material>
+  </gazebo>
+  <gazebo reference="camera_link">
+    <sensor name="camera" type="camera">
+      <always_on>true</always_on>
+      <update_rate>30</update_rate>
+      <topic>camera/image</topic>
+      <camera>
+        <horizontal_fov>2.967</horizontal_fov>  <!-- ~170 degree fisheye -->
+        <image>
+          <width>640</width>
+          <height>480</height>
+          <format>R8G8B8</format>
+        </image>
+        <clip>
+          <near>0.05</near>
+          <far>50.0</far>
+        </clip>
+        <noise>
+          <type>gaussian</type>
+          <mean>0.0</mean>
+          <stddev>0.005</stddev>
+        </noise>
+      </camera>
+    </sensor>
+  </gazebo>
+  <gazebo reference="camera_link">
+    <sensor name="depth_camera" type="depth_camera">
+      <always_on>true</always_on>
+      <update_rate>15</update_rate>
+      <topic>camera/depth</topic>
+      <camera>
+        <horizontal_fov>1.2217</horizontal_fov>  <!-- ~70 degrees for depth -->
+        <image>
+          <width>640</width>
+          <height>480</height>
+          <format>R_FLOAT32</format>
+        </image>
+        <clip>
+          <near>0.1</near>
+          <far>10.0</far>
+        </clip>
+      </camera>
+    </sensor>
+  </gazebo>
+  <!-- ================================================================ -->
+  <!-- 2D LiDAR Sensor — LD06 360° scan for SLAM and navigation         -->
+  <!-- ================================================================ -->
+  <gazebo reference="lidar_link">
+    <material>
+      <ambient>0.2 0.2 0.2 1.0</ambient>
+      <diffuse>0.3 0.3 0.3 1.0</diffuse>
+    </material>
+  </gazebo>
+  <gazebo reference="lidar_link">
+    <sensor name="lidar" type="gpu_lidar">
+      <always_on>true</always_on>
+      <update_rate>10</update_rate>
+      <topic>lidar/scan</topic>
+      <lidar>
+        <scan>
+          <horizontal>
+            <samples>360</samples>
+            <resolution>1</resolution>
+            <min_angle>-3.14159</min_angle>
+            <max_angle>3.14159</max_angle>
+          </horizontal>
+          <vertical>
+            <samples>1</samples>
+            <resolution>1</resolution>
+            <min_angle>0</min_angle>
+            <max_angle>0</max_angle>
+          </vertical>
+        </scan>
+        <range>
+          <min>0.12</min>
+          <max>12.0</max>
+          <resolution>0.01</resolution>
+        </range>
+        <noise>
+          <type>gaussian</type>
+          <mean>0.0</mean>
+          <stddev>0.008</stddev>
+        </noise>
+      </lidar>
+    </sensor>
+  </gazebo>
 </robot>
