File: hardware/pcb/robot-platform.kicad_sch (KiCad schematic)
At the start: 60 parts, among them J1 PBC-34_Payload, J10 Enc_RL, J11 Enc_RR, J2 XT30_Battery, J3 USB-C, J4 Motor_FL, J5 Motor_FR, J6 Motor_RL, J7 Motor_RR, J8 Enc_FL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

Commit message: fix(firmware,ros2,hw): V2 plan P0+P1 critical fixes
P0 — Product-blocking fixes:
- perf(ros2): reuse Hailo InferVStreams pipeline across frames
  Previously opened/closed DMA buffers each frame at 30Hz (<5 FPS).
  Pipeline now opens once at node init, achieving target 25+ FPS.
- hw(pcb): replace SPST safety relay with DPST (Omron G2R-2-H)
  Adds second feedback channel (SAFETY_RELAY_FB2 on GPIO22) with
  independent voltage divider for CE PL d Category 3 compliance.
- feat(firmware): add /charging/voltage Float32 publisher
  Publishes ADC charging pin voltage at 5Hz when docking is enabled,
  unblocking the contact_detector → docking_controller chain.

P1 — Safety and performance:
- feat(ros2): add Ed25519 signature verification to OTA manager
  Uses public_key_path parameter (previously declared but unused).
  Downloads .sig file alongside payload; rejects unsigned updates.
- perf(firmware): separate IMU timer to 100Hz (was 50Hz shared with odom)
  Improves EKF fusion quality with higher-rate orientation data.

Also fixes:
- Remove unused num_classes variable (ruff F841)
- Use color variable in DingTalk notification markdown (ruff F841)
Parts:
- added C15: 100nF, Capacitor_SMD:C_0402_1005Metric, symbol Device:C
- added R13: 20k, Resistor_SMD:R_0603_1608Metric, symbol Device:R
- added R14: 10k, Resistor_SMD:R_0603_1608Metric, symbol Device:R
- RLY1: value Safety_Relay -> G2R-2-H_DC5; footprint Relay_THT:Relay_SPST_Omron_G5V-1 -> Relay_THT:Relay_DPST_Omron_G2R-2; symbol Relay:Relay_SPST -> Relay:Relay_DPST_NO
Changed lines of the file:
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@@
   )
   (symbol
-    (lib_id "Relay:Relay_SPST")
+    (lib_id "Relay:Relay_DPST_NO")
     (at 80 35 0)
-    (property "Reference" "RLY1" (at 80 30 0) (effects (font (size 1.27 1.27))))
-    (property "Value" "Safety_Relay" (at 80 40 0) (effects (font (size 1.27 1.27))))
-    (property "Footprint" "Relay_THT:Relay_SPST_Omron_G5V-1" (at 80 42 0) (effects (font (size 1.27 1.27)) hide))
+    (property "Reference" "RLY1" (at 80 28 0) (effects (font (size 1.27 1.27))))
+    (property "Value" "G2R-2-H_DC5" (at 80 42 0) (effects (font (size 1.27 1.27))))
+    (property "Footprint" "Relay_THT:Relay_DPST_Omron_G2R-2" (at 80 44 0) (effects (font (size 1.27 1.27)) hide))
+    (property "Description" "Dual-channel NO safety relay for CE PL d Category 3" (at 80 46 0) (effects (font (size 1.27 1.27)) hide))
     (pin "1"
     )
@@
     )
     (pin "4"
+    )
+    (pin "5"
+    )
+    (pin "6"
     )
   )
@@
     )
     (pin "GPIO21"
+    )
+    (pin "GPIO22"
     )
     (pin "GPIO26"
@@
   (label "ESTOP" (at 235 92 0) (effects (font (size 1.27 1.27))))
   (label "SAFETY_RELAY_FB" (at 235 95 0) (effects (font (size 1.27 1.27))))
+  (label "SAFETY_RELAY_FB2" (at 235 98 0) (effects (font (size 1.27 1.27))))
   (label "UROS_TX" (at 235 98 0) (effects (font (size 1.27 1.27))))
   (label "UROS_RX" (at 235 101 0) (effects (font (size 1.27 1.27))))
@@
   (label "ESTOP" (at 155 134 0) (effects (font (size 1.27 1.27))))
   (symbol
+    (lib_id "Device:R")
+    (at 175 135 0)
+    (property "Reference" "R13" (at 175 130 0) (effects (font (size 1.27 1.27))))
+    (property "Value" "20k" (at 175 140 0) (effects (font (size 1.27 1.27))))
+    (property "Footprint" "Resistor_SMD:R_0603_1608Metric" (at 175 142 0) (effects (font (size 1.27 1.27)) hide))
+    (property "Description" "Relay FB2 voltage divider upper" (at 175 144 0) (effects (font (size 1.27 1.27)) hide))
+    (pin "1"
+    )
+    (pin "2"
+    )
+  )
+  (symbol
+    (lib_id "Device:R")
+    (at 175 148 0)
+    (property "Reference" "R14" (at 175 143 0) (effects (font (size 1.27 1.27))))
+    (property "Value" "10k" (at 175 153 0) (effects (font (size 1.27 1.27))))
+    (property "Footprint" "Resistor_SMD:R_0603_1608Metric" (at 175 155 0) (effects (font (size 1.27 1.27)) hide))
+    (property "Description" "Relay FB2 voltage divider lower" (at 175 157 0) (effects (font (size 1.27 1.27)) hide))
+    (pin "1"
+    )
+    (pin "2"
+    )
+  )
+  (symbol
+    (lib_id "Device:C")
+    (at 185 148 0)
+    (property "Reference" "C15" (at 185 143 0) (effects (font (size 1.27 1.27))))
+    (property "Value" "100nF" (at 185 153 0) (effects (font (size 1.27 1.27))))
+    (property "Footprint" "Capacitor_SMD:C_0402_1005Metric" (at 185 155 0) (effects (font (size 1.27 1.27)) hide))
+    (property "Description" "Relay FB2 RC filter" (at 185 157 0) (effects (font (size 1.27 1.27)) hide))
+    (pin "1"
+    )
+    (pin "2"
+    )
+  )
+  (label "VBAT_MOTOR" (at 175 128 0) (effects (font (size 1.27 1.27))))
+  (label "SAFETY_RELAY_FB2" (at 183 142 0) (effects (font (size 1.27 1.27))))
+  (symbol
+    (lib_id "power:GND")
+    (at 175 155 0)
+    (property "Reference" "#PWR32" (at 175 153 0) (effects (font (size 1.27 1.27)) hide))
+    (property "Value" "GND" (at 175 157 0) (effects (font (size 1.27 1.27))))
+    (pin "1"
+    )
+  )
+  (symbol
     (lib_id "Connector:USB_C_Receptacle_USB2.0")
     (at 160 245 0)
@@
       (reference "RLY1")
       (unit 1)
-      (value "Safety_Relay")
+      (value "G2R-2-H_DC5")
       (footprint "")
     )

Commit message: feat(firmware,hardware): align dock detection spec + add 12V P-MOS switch with extensible power rail abstraction
Issue 1 — Dock detection method alignment:
- Update hardware spec: Pin 1 is dual-purpose (charge sense + ADC dock
  detection), Pin 4 marked RESERVED for future use
- Add Kconfig option CONFIG_ROBOT_DOCKING_DIGITAL_DETECT for optional
  secondary digital GPIO detection (OR-logic with analog)
- Extend charging_detect module with charge_detect_method_t enum and
  charging_detect_get_method() API

Issue 2 — 12V payload power rail P-MOS high-side switch:
- Add AO3401A (Q4) circuit to KiCad schematic (Vds=-30V, Id=-4A, SOT-23)
  with R16 100k gate pull-up, matching Q3 (5V) topology
- Create payload_power.h/c: generic power rail controller supporting up to
  4 rails with configurable soft-start, overcurrent thresholds, per-rail
  state machine (OFF/RAMPING/ON/FAULT)
- Extract mcp23017_write_bit() and mcp23017_read_register() to shared
  i2c_bus module for reuse across payload_hotplug and payload_power
- Refactor payload_hotplug.c to use shared I2C utility

Extensibility:
- Future rails (24V, variable) need only a config entry + hardware switch
- Future dock revisions can use digital detect via Kconfig toggle
- Power rail module is independent of hotplug state machine

Also fixes pre-existing test build issues:
- Add missing ADC_CHANNEL_4-7 definitions to test stubs
- Add CONFIG_ROBOT_DUAL_BATTERY to test Makefile CFLAGS

285 tests pass, 0 failures.
Parts:
- added Q3: Si2301CDS, Package_TO_SOT_SMD:SOT-23, symbol Transistor_FET:Si2301CDS
- added Q4: AO3401A, Package_TO_SOT_SMD:SOT-23, symbol Transistor_FET:AO3401A
- added R15, R16: 100k, Resistor_SMD:R_0402_1005Metric, symbol Device:R
Changed lines of the file:
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@@
   (label "ENC_RR_A" (at 165 71 0) (effects (font (size 1.27 1.27))))
   (label "US_ECHO_LEFT" (at 165 74 0) (effects (font (size 1.27 1.27))))
+  (label "CAN_INT" (at 165 74 0) (effects (font (size 1.27 1.27))))
   (label "US_ECHO_BACK" (at 165 77 0) (effects (font (size 1.27 1.27))))
+  (label "CAN_MISO" (at 165 77 0) (effects (font (size 1.27 1.27))))
   (label "US_ECHO_FRONT" (at 165 80 0) (effects (font (size 1.27 1.27))))
+  (label "CAN_MOSI" (at 165 80 0) (effects (font (size 1.27 1.27))))
   (label "US_TRIG" (at 165 83 0) (effects (font (size 1.27 1.27))))
+  (label "CAN_SCLK" (at 165 83 0) (effects (font (size 1.27 1.27))))
   (label "MOT_FL_IN1" (at 165 86 0) (effects (font (size 1.27 1.27))))
   (label "MOT_FL_IN2" (at 165 89 0) (effects (font (size 1.27 1.27))))
@@
   (label "ENC_RL_B" (at 235 56 0) (effects (font (size 1.27 1.27))))
   (label "US_ECHO_RIGHT" (at 235 59 0) (effects (font (size 1.27 1.27))))
+  (label "CAN_CS" (at 235 59 0) (effects (font (size 1.27 1.27))))
   (label "MOT_FR_IN1" (at 235 65 0) (effects (font (size 1.27 1.27))))
-  (label "CAN_INT" (at 235 68 0) (effects (font (size 1.27 1.27))))
-  (label "CAN_CS" (at 235 71 0) (effects (font (size 1.27 1.27))))
-  (label "CAN_MOSI" (at 235 74 0) (effects (font (size 1.27 1.27))))
-  (label "CAN_SCLK" (at 235 77 0) (effects (font (size 1.27 1.27))))
-  (label "CAN_MISO" (at 235 80 0) (effects (font (size 1.27 1.27))))
+  (label "SAFETY_RELAY_FB2" (at 235 68 0) (effects (font (size 1.27 1.27))))
   (label "MOT_RL_IN2" (at 235 83 0) (effects (font (size 1.27 1.27))))
   (label "MOT_RR_IN1" (at 235 86 0) (effects (font (size 1.27 1.27))))
@@
   (label "ESTOP" (at 235 92 0) (effects (font (size 1.27 1.27))))
   (label "SAFETY_RELAY_FB" (at 235 95 0) (effects (font (size 1.27 1.27))))
-  (label "SAFETY_RELAY_FB2" (at 235 98 0) (effects (font (size 1.27 1.27))))
   (label "UROS_TX" (at 235 98 0) (effects (font (size 1.27 1.27))))
   (label "UROS_RX" (at 235 101 0) (effects (font (size 1.27 1.27))))
@@
   (label "PAYLOAD_ENABLE" (at 325 188 0) (effects (font (size 1.27 1.27))))
   (label "PAYLOAD_FAULT" (at 325 191 0) (effects (font (size 1.27 1.27))))
-  (label "PAYLOAD_DETECT" (at 325 194 0) (effects (font (size 1.27 1.27))))
+  (label "PBC_DETECT" (at 325 194 0) (effects (font (size 1.27 1.27))))
   (label "PAYLOAD_INT" (at 325 197 0) (effects (font (size 1.27 1.27))))
   (label "+3V3" (at 325 200 0) (effects (font (size 1.27 1.27))))
@@
     )
   )
+  (symbol
+    (lib_id "Transistor_FET:Si2301CDS")
+    (at 290 165 0)
+    (mirror y)
+    (property "Reference" "Q3" (at 290 160 0) (effects (font (size 1.27 1.27))))
+    (property "Value" "Si2301CDS" (at 290 170 0) (effects (font (size 1.27 1.27))))
+    (property "Footprint" "Package_TO_SOT_SMD:SOT-23" (at 290 172 0) (effects (font (size 1.27 1.27)) hide))
+    (property "Description" "Payload 5V power switch (P-MOS, controlled by PBC_5V_EN via MCP23017)" (at 290 174 0) (effects (font (size 1.27 1.27)) hide))
+    (pin "G"
+    )
+    (pin "S"
+    )
+    (pin "D"
+    )
+  )
+  (label "+5V_ESP" (at 285 162 0) (effects (font (size 1.27 1.27))))
+  (label "+5V_PAYLOAD" (at 295 162 0) (effects (font (size 1.27 1.27))))
+  (label "PBC_5V_EN" (at 290 172 0) (effects (font (size 1.27 1.27))))
+  (symbol
+    (lib_id "Device:R")
+    (at 290 175 0)
+    (property "Reference" "R15" (at 290 170 0) (effects (font (size 1.27 1.27))))
+    (property "Value" "100k" (at 290 180 0) (effects (font (size 1.27 1.27))))
+    (property "Footprint" "Resistor_SMD:R_0402_1005Metric" (at 290 182 0) (effects (font (size 1.27 1.27)) hide))
+    (property "Description" "P-MOS gate pull-up (default OFF)" (at 290 184 0) (effects (font (size 1.27 1.27)) hide))
+    (pin "1"
+    )
+    (pin "2"
+    )
+  )
+  (label "+5V_ESP" (at 290 179 0) (effects (font (size 1.27 1.27))))
+  (symbol
+    (lib_id "Transistor_FET:AO3401A")
+    (at 310 165 0)
+    (mirror y)
+    (property "Reference" "Q4" (at 310 160 0) (effects (font (size 1.27 1.27))))
+    (property "Value" "AO3401A" (at 310 170 0) (effects (font (size 1.27 1.27))))
+    (property "Footprint" "Package_TO_SOT_SMD:SOT-23" (at 310 172 0) (effects (font (size 1.27 1.27)) hide))
+    (property "Description" "Payload 12V power switch (P-MOS, Vds=-30V Id=-4A, controlled by PBC_12V_EN via MCP23017)" (at 310 174 0) (effects (font (size 1.27 1.27)) hide))
+    (pin "G"
+    )
+    (pin "S"
+    )
+    (pin "D"
+    )
+  )
+  (label "+12V_BOOST" (at 305 162 0) (effects (font (size 1.27 1.27))))
+  (label "+12V_PAYLOAD" (at 315 162 0) (effects (font (size 1.27 1.27))))
+  (label "PBC_12V_EN" (at 310 172 0) (effects (font (size 1.27 1.27))))
+  (symbol
+    (lib_id "Device:R")
+    (at 310 175 0)
+    (property "Reference" "R16" (at 310 170 0) (effects (font (size 1.27 1.27))))
+    (property "Value" "100k" (at 310 180 0) (effects (font (size 1.27 1.27))))
+    (property "Footprint" "Resistor_SMD:R_0402_1005Metric" (at 310 182 0) (effects (font (size 1.27 1.27)) hide))
+    (property "Description" "12V P-MOS gate pull-up (default OFF)" (at 310 184 0) (effects (font (size 1.27 1.27)) hide))
+    (pin "1"
+    )
+    (pin "2"
+    )
+  )
+  (label "+12V_BOOST" (at 310 179 0) (effects (font (size 1.27 1.27))))
   (text "POWER SUPPLY" (at 60 12 0) (effects (font (size 3 3) bold)))
   (text "MCU - ESP32-S3" (at 200 15 0) (effects (font (size 3 3) bold)))

Commit message: hw(pcb): fix critical hardware design issues for production readiness
Fix 1: Replace MT3608 boost (wrong topology) with MP2359DJ buck converter
  - VBAT 7.4V → 5V is a step-down, not step-up operation
  - Add feedback divider R30/R31 (44.2k/10k for 5.0V output)
  - Change inductor L1 from 4.7uH to 10uH for buck operation

Fix 2: Add HC-SR04 echo 5V→3.3V level shift (R20-R27)
  - 4× resistive divider (10k series + 18k shunt) per echo channel
  - Prevents 5V echo signal from damaging ESP32-S3 GPIO

Fix 3: Add safety relay driver circuit
  - Q5 (AO3400A N-MOS) for relay coil low-side drive
  - D5 (1N4148W) flyback protection across coil
  - R17/R18 gate bias (hardware interlock, not software-controlled)

Fix 4: Add DRV8833 nSLEEP external pull-ups (R28-R29)
  - 10k to +3V3 on both motor drivers
  - Prevents EMI-induced sleep entry in vibration environments

Fix 5: Reduce TP5100 charge current from 2A to 1.5A
  - R6 changed from 1.2kΩ to 1.5kΩ
  - Thermal dissipation reduced from 7.2W to 5.4W

Fix 6: Replace AMS1117-3.3 (SOT-223) with AP2112K-3.3 (SOT-23-5)
  - Dropout reduced from 1.3V to 250mV
  - Better thermal performance at equivalent load

BOM corrected to match schematic reality:
- R9 = 120Ω CAN termination (not ultrasonic)
- R10-R11 = 5.1k USB-C CC (not ultrasonic)
- Individual references for all new components

All validation scripts pass:
- validate_hardware.py: PASS
- validate-pin-conflicts.py: PASS
- validate-bom-firmware.py: PASS

Schematic rev bumped: 1.0 → 1.1
Parts:
- added D5: 1N4148W, Diode_SMD:D_SOD-123, symbol Diode:1N4148W
- added Q5: AO3400A, Package_TO_SOT_SMD:SOT-23, symbol Transistor_FET:AO3400A
- added R17, R20, R22, R24, R26, R28, R29: 10k, Resistor_SMD:R_0402_1005Metric, symbol Device:R
- added R18: 100k, Resistor_SMD:R_0402_1005Metric, symbol Device:R
- added R21, R23, R25, R27: 18k, Resistor_SMD:R_0402_1005Metric, symbol Device:R
- added R30: 44.2k 1%, Resistor_SMD:R_0402_1005Metric, symbol Device:R
- added R31: 10k 1%, Resistor_SMD:R_0402_1005Metric, symbol Device:R
- U3: value AMS1117-3.3 -> AP2112K-3.3; footprint Package_TO_SOT_SMD:SOT-223-3_TabPin2 -> Package_TO_SOT_SMD:SOT-23-5; symbol Regulator_Linear:AMS1117-3.3 -> Regulator_Linear:AP2112K-3.3
- U4: value MT3608_5V_ESP -> MP2359DJ_5V_ESP; footprint Package_SO:SOT-23-6 -> Package_TO_SOT_SMD:SOT-23-6; symbol Regulator_Switching:MT3608 -> Regulator_Switching:MP2359
Other:
- note added: "RELAY DRIVER"
- note added: "US ECHO LEVEL SHIFT"

Commit message: hw(pcb): fix payload 5V overload, nFAULT monitoring, TP5100 thermal, CAN docs
Fix 7: Move Payload 5V source from +5V_ESP (1.2A) to +5V_PI (5A)
  - Q3 Si2301CDS source net changed to +5V_PI
  - R15 gate pull-up also moved to +5V_PI rail
  - Prevents MP2359 overload when payload draws >500mA
  - PBC-34 pin 1-2 documentation updated

Fix 8: Add DRV8833 nFAULT monitoring (R32/R33)
  - 10k pull-ups on open-drain nFAULT outputs
  - Routed to MCP23017 GPB4/GPB5 for firmware detection
  - Enables overcurrent and thermal fault awareness

Fix 9: TP5100 charge current reduced to 1.0A (R6=2.4kΩ)
  - 12V input dissipation: 3.6W (safe with 1.5cm² copper)
  - 9V USB-C PD input: 0.6W (preferred operation)
  - Charge time ~3h for 3000mAh (acceptable)

Fix 10: CAN termination resistor R9 documentation
  - Added explicit population rules in PCB README
  - Added R9 to Industrial BOM with topology guidance

All validation scripts pass (3/3).
Parts:
- added R32, R33: 10k, Resistor_SMD:R_0402_1005Metric, symbol Device:R
Changed lines of the file:
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@@
   (label "+3V3" (at 325 58 0) (effects (font (size 1.27 1.27))))
+  (symbol
+    (lib_id "Device:R")
+    (at 335 32 0)
+    (property "Reference" "R32" (at 335 27 0) (effects (font (size 1.27 1.27))))
+    (property "Value" "10k" (at 335 37 0) (effects (font (size 1.27 1.27))))
+    (property "Footprint" "Resistor_SMD:R_0402_1005Metric" (at 335 39 0) (effects (font (size 1.27 1.27)) hide))
+    (property "Description" "DRV8833_Front nFAULT pull-up (open-drain output)" (at 335 41 0) (effects (font (size 1.27 1.27)) hide))
+    (pin "1"
+    )
+    (pin "2"
+    )
+  )
+  (label "+3V3" (at 335 25 0) (effects (font (size 1.27 1.27))))
+  (label "DRV_FAULT_FRONT" (at 340 37 0) (effects (font (size 1.27 1.27))))
+  (symbol
+    (lib_id "Device:R")
+    (at 335 72 0)
+    (property "Reference" "R33" (at 335 67 0) (effects (font (size 1.27 1.27))))
+    (property "Value" "10k" (at 335 77 0) (effects (font (size 1.27 1.27))))
+    (property "Footprint" "Resistor_SMD:R_0402_1005Metric" (at 335 79 0) (effects (font (size 1.27 1.27)) hide))
+    (property "Description" "DRV8833_Rear nFAULT pull-up (open-drain output)" (at 335 81 0) (effects (font (size 1.27 1.27)) hide))
+    (pin "1"
+    )
+    (pin "2"
+    )
+  )
+  (label "+3V3" (at 335 65 0) (effects (font (size 1.27 1.27))))
+  (label "DRV_FAULT_REAR" (at 340 77 0) (effects (font (size 1.27 1.27))))
   (symbol
     (lib_id "Device:C")
@@
   (label "PBC_GPIO6" (at 225 198 0) (effects (font (size 1.27 1.27))))
   (label "PBC_GPIO7" (at 225 201 0) (effects (font (size 1.27 1.27))))
+  (label "DRV_FAULT_FRONT" (at 225 204 0) (effects (font (size 1.27 1.27))))
+  (label "DRV_FAULT_REAR" (at 225 207 0) (effects (font (size 1.27 1.27))))
   (symbol
     (lib_id "Device:C")
@@
     )
   )
-  (label "+5V_ESP" (at 285 162 0) (effects (font (size 1.27 1.27))))
+  (label "+5V_PI" (at 285 162 0) (effects (font (size 1.27 1.27))))
   (label "+5V_PAYLOAD" (at 295 162 0) (effects (font (size 1.27 1.27))))
   (label "PBC_5V_EN" (at 290 172 0) (effects (font (size 1.27 1.27))))
@@
     )
   )
-  (label "+5V_ESP" (at 290 179 0) (effects (font (size 1.27 1.27))))
+  (label "+5V_PI" (at 290 179 0) (effects (font (size 1.27 1.27))))
   (symbol
     (lib_id "Transistor_FET:AO3401A")

Commit message: hw(pcb): add TPS3813 watchdog, Pi5 power switch, fix INA219 shunt, BNO055 cap, MCP INT
Fix 11: Q4/R16 marked DNP on Basic SKU (no +12V_BOOST source)
Fix 12: TPS3813K33DBVR external watchdog (GPIO46 WDI, 1.6s timeout → ESP32 EN reset)
Fix 13: Pi5 power switch (dual Si2301CDS + AO3400A, GPIO45, Standard/Industrial only)
Fix 14: R7 shunt 0.1Ω → 0.02Ω (INA219 calibration updated, 0.5W@5A vs prior 2.5W)
Fix 15: C17 10µF bulk cap on BNO055 VDD (per datasheet recommendation)
Fix 16: R36 10k pull-up on MCP23017 INTA + TP1 test pad

Schematic bumped to Rev 1.1c. All validation scripts pass (289 firmware tests OK).
Parts:
- added C16: 100nF, Capacitor_SMD:C_0402_1005Metric, symbol Device:C
- added C17: 10uF, Capacitor_SMD:C_0805_2012Metric, symbol Device:C
- added Q6a, Q6b: Si2301CDS, Package_TO_SOT_SMD:SOT-23, symbol Transistor_FET:Si2301CDS
- added Q7: AO3400A, Package_TO_SOT_SMD:SOT-23, symbol Transistor_FET:AO3400A
- added R34, R35: 100k, Resistor_SMD:R_0402_1005Metric, symbol Device:R
- added R36: 10k, Resistor_SMD:R_0402_1005Metric, symbol Device:R
- added TP1: MCP_INTA, TestPoint:TestPoint_Pad_1.0x1.0mm, symbol Connector:TestPoint
- added U10: TPS3813K33DBVR, Package_TO_SOT_SMD:SOT-23-5, symbol Timer:TPS3813
- R7: value 0.1R -> 0.02R
Other:
- note added: "BNO055 BULK CAP"
- note added: "EXTERNAL WATCHDOG"
- note added: "MCP23017 INT"
- note added: "PI5 POWER SWITCH"
