File: hardware/pcb/robot-platform.kicad_sch (KiCad schematic)
At the start: 102 parts, among them J1 PBC-34_Payload, J10 Enc_RL, J11 Enc_RR, J2 XT30_Battery, J3 USB-C, J4 Motor_FL, J5 Motor_FR, J6 Motor_RL, J7 Motor_RR, J8 Enc_FL, J9 Enc_FR, Q3 Si2301CDS, Q4 AO3401A, Q5 AO3400A, Q6a Si2301CDS, Q6b Si2301CDS, Q7 AO3400A, Q8a AO3401A, Q8b AO3401A, SW1 E-STOP_NC, SW1b E-STOP_NC2, U1 ESP32-S3-WROOM-1-N8R8, U10 TPS3813K33DBVR, U2a DRV8833_Front, U2b DRV8833_Rear, U3 AP2112K-3.3, U4 MP2359DJ_5V_ESP, U5 MP1584EN_5V_PI, U6 MCP23017-E/SO, U7 INA219BIDR, U8 MCP2515, U9 TJA1050, Y1 8MHz

Commit message: hw(hardware): fixes 32-37 — buck Schottky/BST, E-stop polarity, I2C addr, USB ESD
Fix 32: Add SS34 Schottky diode (D6) and bootstrap cap (C19) for MP2359
Fix 33: Add SS54 Schottky diode (D7) and bootstrap cap (C20) for MP1584EN
Fix 34: Invert E-stop polarity — SW1 passes +3V3 via NC, R5 pulls down
         (ISO 13850 fail-safe: wire break → ESTOP=LOW → safe state)
Fix 35: Tie BNO055 PS0/PS1/ADR to GND (I2C mode, addr 0x28)
Fix 36: Add USBLC6-2SC6 (U11) USB ESD protection on D+/D-
Fix 37: Tie MCP23017 A0/A1/A2 to GND (addr 0x20)

Schematic bumped to Rev 1.1f. All validations pass (pin conflicts,
BOM-firmware alignment, hardware validation). 289 firmware tests pass.

BOM delta: +¥1.44/board (D6, D7, C19, C20, U11)
Parts:
- added C19, C20: 100nF, Capacitor_SMD:C_0402_1005Metric, symbol Device:C
- added D6: SS34, Diode_SMD:D_SOD-123F, symbol Diode:SS34
- added D7: SS54, Diode_SMD:D_SMA, symbol Diode:SS54
- added U11: USBLC6-2SC6, Package_TO_SOT_SMD:SOT-23-6, symbol Power_Protection:USBLC6-2SC6
Changed lines of the file:
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@@
     (comment 1 "SPDX-License-Identifier: CERN-OHL-P-2.0")
     (comment 2 "Universal Modular Mobile Platform")
-    (comment 3 "Rev 1.1e: E-stop hardwire relay, DRV8833 xISEN GND, nSLEEP→ESTOP, safety architecture")
+    (comment 3 "Rev 1.1f: Buck Schottky/BST caps, E-stop polarity fix, I2C addr ties, USB ESD")
   )
   (symbol
@@
     (property "Value" "MP2359DJ_5V_ESP" (at 50 65 0) (effects (font (size 1.27 1.27))))
     (property "Footprint" "Package_TO_SOT_SMD:SOT-23-6" (at 50 67 0) (effects (font (size 1.27 1.27)) hide))
-    (property "Description" "5V/1.2A synchronous buck converter (VBAT 7.4V input)" (at 50 69 0) (effects (font (size 1.27 1.27)) hide))
+    (property "Description" "5V/1.2A asynchronous buck converter (VBAT 7.4V input, external Schottky D6)" (at 50 69 0) (effects (font (size 1.27 1.27)) hide))
     (pin "IN"
     )
@@
     )
   )
+  (label "MP2359_SW" (at 55 62 0) (effects (font (size 1.27 1.27))))
+  (symbol
+    (lib_id "Diode:SS34")
+    (at 55 68 270)
+    (property "Reference" "D6" (at 58 68 0) (effects (font (size 1.27 1.27))))
+    (property "Value" "SS34" (at 55 71 0) (effects (font (size 1.27 1.27))))
+    (property "Footprint" "Diode_SMD:D_SOD-123F" (at 55 73 0) (effects (font (size 1.27 1.27)) hide))
+    (property "Description" "MP2359 freewheeling Schottky diode (cathode=SW, anode=GND). 40V/3A." (at 55 75 0) (effects (font (size 1.27 1.27)) hide))
+    (pin "K"
+    )
+    (pin "A"
+    )
+  )
+  (label "MP2359_SW" (at 55 65 0) (effects (font (size 1.27 1.27))))
+  (symbol
+    (lib_id "power:GND")
+    (at 55 72 0)
+    (property "Reference" "#PWR45" (at 55 74 0) (effects (font (size 1.27 1.27)) hide))
+    (property "Value" "GND" (at 55 76 0) (effects (font (size 1.27 1.27))))
+    (pin "1"
+    )
+  )
+  (symbol
+    (lib_id "Device:C")
+    (at 45 58 0)
+    (property "Reference" "C19" (at 45 54 0) (effects (font (size 1.27 1.27))))
+    (property "Value" "100nF" (at 45 62 0) (effects (font (size 1.27 1.27))))
+    (property "Footprint" "Capacitor_SMD:C_0402_1005Metric" (at 45 64 0) (effects (font (size 1.27 1.27)) hide))
+    (property "Description" "MP2359 bootstrap capacitor (BST to SW)" (at 45 66 0) (effects (font (size 1.27 1.27)) hide))
+    (pin "1"
+    )
+    (pin "2"
+    )
+  )
+  (label "MP2359_BST" (at 45 55 0) (effects (font (size 1.27 1.27))))
+  (label "MP2359_SW" (at 45 62 0) (effects (font (size 1.27 1.27))))
   (symbol
     (lib_id "Regulator_Switching:MP1584EN")
@@
     )
   )
+  (label "MP1584_SW" (at 55 92 0) (effects (font (size 1.27 1.27))))
+  (symbol
+    (lib_id "Diode:SS54")
+    (at 55 97 270)
+    (property "Reference" "D7" (at 58 97 0) (effects (font (size 1.27 1.27))))
+    (property "Value" "SS54" (at 55 100 0) (effects (font (size 1.27 1.27))))
+    (property "Footprint" "Diode_SMD:D_SMA" (at 55 102 0) (effects (font (size 1.27 1.27)) hide))
+    (property "Description" "MP1584EN freewheeling Schottky diode (cathode=SW, anode=GND). 40V/5A." (at 55 104 0) (effects (font (size 1.27 1.27)) hide))
+    (pin "K"
+    )
+    (pin "A"
+    )
+  )
+  (label "MP1584_SW" (at 55 94 0) (effects (font (size 1.27 1.27))))
+  (symbol
+    (lib_id "power:GND")
+    (at 55 101 0)
+    (property "Reference" "#PWR46" (at 55 103 0) (effects (font (size 1.27 1.27)) hide))
+    (property "Value" "GND" (at 55 105 0) (effects (font (size 1.27 1.27))))
+    (pin "1"
+    )
+  )
+  (symbol
+    (lib_id "Device:C")
+    (at 45 88 0)
+    (property "Reference" "C20" (at 45 84 0) (effects (font (size 1.27 1.27))))
+    (property "Value" "100nF" (at 45 92 0) (effects (font (size 1.27 1.27))))
+    (property "Footprint" "Capacitor_SMD:C_0402_1005Metric" (at 45 94 0) (effects (font (size 1.27 1.27)) hide))
+    (property "Description" "MP1584EN bootstrap capacitor (BST to SW)" (at 45 96 0) (effects (font (size 1.27 1.27)) hide))
+    (pin "1"
+    )
+    (pin "2"
+    )
+  )
+  (label "MP1584_BST" (at 45 85 0) (effects (font (size 1.27 1.27))))
+  (label "MP1584_SW" (at 45 92 0) (effects (font (size 1.27 1.27))))
   (symbol
     (lib_id "Regulator_Linear:AP2112K-3.3")
@@
     )
   )
+  (symbol
+    (lib_id "power:GND")
+    (at 65 218 0)
+    (property "Reference" "#PWR47" (at 65 220 0) (effects (font (size 1.27 1.27)) hide))
+    (property "Value" "GND" (at 65 222 0) (effects (font (size 1.27 1.27))))
+    (property "Description" "BNO055 PS0/PS1/ADR tied to GND (selects I2C mode, address 0x28)" (at 65 224 0) (effects (font (size 1.27 1.27)) hide))
+    (pin "1"
+    )
+  )
   (label "I2C_SDA" (at 30 200 0) (effects (font (size 1.27 1.27))))
   (label "I2C_SCL" (at 30 203 0) (effects (font (size 1.27 1.27))))
@@
     )
     (pin "A2"
+    )
+  )
+  (symbol
+    (lib_id "power:GND")
+    (at 180 195 0)
+    (property "Reference" "#PWR49" (at 180 197 0) (effects (font (size 1.27 1.27)) hide))
+    (property "Value" "GND" (at 180 199 0) (effects (font (size 1.27 1.27))))
+    (property "Description" "MCP23017 A0/A1/A2 tied to GND (I2C address = 0x20)" (at 180 201 0) (effects (font (size 1.27 1.27)) hide))
+    (pin "1"
     )
   )
@@
   (label "ESTOP" (at 155 135 0) (effects (font (size 1.27 1.27))))
   (symbol
-    (lib_id "power:GND")
+    (lib_id "power:+3V3")
     (at 135 135 0)
     (property "Reference" "#PWR28" (at 135 133 0) (effects (font (size 1.27 1.27)) hide))
-    (property "Value" "GND" (at 135 137 0) (effects (font (size 1.27 1.27))))
+    (property "Value" "+3V3" (at 135 131 0) (effects (font (size 1.27 1.27))))
+    (property "Description" "SW1 NC contact source — E-stop NC passes 3.3V to ESTOP net (fail-safe: wire break → pull-down → LOW → safe)" (at 135 139 0) (effects (font (size 1.27 1.27)) hide))
     (pin "1"
     )
@@
     )
   )
-  (label "+3V3" (at 155 122 0) (effects (font (size 1.27 1.27))))
+  (label "GND" (at 155 122 0) (effects (font (size 1.27 1.27))))
   (label "ESTOP" (at 155 134 0) (effects (font (size 1.27 1.27))))
   (symbol
@@
   (label "USB_DP" (at 180 240 0) (effects (font (size 1.27 1.27))))
   (label "USB_DN" (at 180 243 0) (effects (font (size 1.27 1.27))))
+  (symbol
+    (lib_id "Power_Protection:USBLC6-2SC6")
+    (at 185 250 0)
+    (property "Reference" "U11" (at 185 244 0) (effects (font (size 1.27 1.27))))
+    (property "Value" "USBLC6-2SC6" (at 185 256 0) (effects (font (size 1.27 1.27))))
+    (property "Footprint" "Package_TO_SOT_SMD:SOT-23-6" (at 185 258 0) (effects (font (size 1.27 1.27)) hide))
+    (property "Description" "USB D+/D- ESD protection (±15kV air, ±8kV contact, IEC 61000-4-2)" (at 185 260 0) (effects (font (size 1.27 1.27)) hide))
+    (pin "1"
+    )
+    (pin "2"
+    )
+    (pin "3"
+    )
+    (pin "4"
+    )
+    (pin "5"
+    )
+    (pin "6"
+    )
+  )
+  (label "USB_DP" (at 185 247 0) (effects (font (size 1.27 1.27))))
+  (label "USB_DN" (at 185 253 0) (effects (font (size 1.27 1.27))))
+  (label "+5V_USB" (at 190 244 0) (effects (font (size 1.27 1.27))))
+  (symbol
+    (lib_id "power:GND")
+    (at 185 258 0)
+    (property "Reference" "#PWR48" (at 185 260 0) (effects (font (size 1.27 1.27)) hide))
+    (property "Value" "GND" (at 185 262 0) (effects (font (size 1.27 1.27))))
+    (pin "1"
+    )
+  )
   (symbol
     (lib_id "power:GND")
@@
       (reference "#PWR28")
       (unit 1)
-      (value "GND")
+      (value "+3V3")
       (footprint "")
     )
@@
       (unit 1)
       (value "GND")
+      (footprint "")
+    )
+    (path "/a1b2c3d4-0032-0002-0001-000000000001"
+      (reference "D6")
+      (unit 1)
+      (value "SS34")
+      (footprint "Diode_SMD:D_SOD-123F")
+    )
+    (path "/a1b2c3d4-0032-0004-0001-000000000001"
+      (reference "#PWR45")
+      (unit 1)
+      (value "GND")
+      (footprint "")
+    )
+    (path "/a1b2c3d4-0032-0005-0001-000000000001"
+      (reference "C19")
+      (unit 1)
+      (value "100nF")
+      (footprint "Capacitor_SMD:C_0402_1005Metric")
+    )
+    (path "/a1b2c3d4-0033-0002-0001-000000000001"
+      (reference "D7")
+      (unit 1)
+      (value "SS54")
+      (footprint "Diode_SMD:D_SMA")
+    )
+    (path "/a1b2c3d4-0033-0004-0001-000000000001"
+      (reference "#PWR46")
+      (unit 1)
+      (value "GND")
+      (footprint "")
+    )
+    (path "/a1b2c3d4-0033-0005-0001-000000000001"
+      (reference "C20")
+      (unit 1)
+      (value "100nF")
+      (footprint "Capacitor_SMD:C_0402_1005Metric")
+    )
+    (path "/a1b2c3d4-0035-0001-0001-000000000001"
+      (reference "#PWR47")
+      (unit 1)
+      (value "GND")
+      (footprint "")
+    )
+    (path "/a1b2c3d4-0036-0001-0001-000000000001"
+      (reference "U11")
+      (unit 1)
+      (value "USBLC6-2SC6")
+      (footprint "Package_TO_SOT_SMD:SOT-23-6")
+    )
+    (path "/a1b2c3d4-0036-0005-0001-000000000001"
+      (reference "#PWR48")
+      (unit 1)
+      (value "GND")
+      (footprint "")
+    )
+    (path "/a1b2c3d4-0037-0001-0001-000000000001"
+      (reference "#PWR49")
+      (unit 1)
+      (value "GND")
